File: hardware/kicad/jjy-hat.kicad_sch (KiCad schematic)
At the start: 26 parts, among them J1 GPIO 2x20 stacking header, J2 Antenna, K1 AQY212SX, U1 74LVC125, U2 DS3231SN#

Commit message: Rev C board: LCD, LEDs, PCB spiral antenna, antenna select, optional resonance
- Leaded R/LED/C parts (hand-soldered); only U1/U2 are SMT at JLCPCB
- 16x2 I2C LCD (J3) shows current time; signal LED (low-level period),
  level LED and power pilot LED grouped at the board's top-left
- Antenna is an on-board PCB spiral coil; JP1 selects it or external J2
- Optional (DNP) resonance bank + K1 40/60kHz switch for external coils
- J1 at top-center, board 100x96 mm to fit the metal case via a cable
- jjyd: LCD driver, signal LED, optional select_gpio, DS3231 RTC support
- Regenerated Gerber/BOM/CPL and updated docs

Co-Authored-By: Claude Sonnet 5.5 <noreply@anthropic.com>
Parts:
- added D2: LED green, LED_THT:LED_D3.0mm, symbol Device:LED
- added D3: LED yellow, LED_THT:LED_D3.0mm, symbol Device:LED
- added J3: I2C LCD (AE-AQM1602A), Connector_PinSocket_2.54mm:PinSocket_1x04_P2.54mm_Vertical, symbol Connector_Generic:Conn_01x04
- added JP1: Antenna select, Connector_PinHeader_2.54mm:PinHeader_1x03_P2.54mm_Vertical, symbol Connector_Generic:Conn_01x03
- added JP2: Resonance bypass, Connector_PinHeader_2.54mm:PinHeader_1x02_P2.54mm_Vertical, symbol Connector_Generic:Conn_01x02
- added L1: PCB spiral coil, JJY:Coil_Spiral, symbol Device:L
- added R7: 330, Resistor_THT:R_Axial_DIN0207_L6.3mm_D2.5mm_P2.54mm_Vertical, symbol Device:R
- added R8: 470, Resistor_THT:R_Axial_DIN0207_L6.3mm_D2.5mm_P2.54mm_Vertical, symbol Device:R
- C1, C5, C6: footprint Capacitor_SMD:C_0603_1608Metric -> Capacitor_THT:C_Rect_L7.0mm_W2.0mm_P5.00mm
- C2, C7: value 4.7n C0G -> 4.7n C0G (DNP); footprint Capacitor_SMD:C_0603_1608Metric -> Capacitor_THT:C_Rect_L7.0mm_W2.0mm_P5.00mm; now not fitted
- C3, C8, C9: value 2.2n C0G -> 2.2n C0G (DNP); footprint Capacitor_SMD:C_0603_1608Metric -> Capacitor_THT:C_Rect_L7.0mm_W2.0mm_P5.00mm; now not fitted
- C4: value 150p C0G -> 150p C0G (DNP); footprint Capacitor_SMD:C_0603_1608Metric -> Capacitor_THT:C_Rect_L7.0mm_W2.0mm_P5.00mm; now not fitted
- D1: footprint LED_SMD:LED_0603_1608Metric -> LED_THT:LED_D3.0mm
- J1: value GPIO 2x20 stacking header -> GPIO 2x20 pin header (ribbon / Dupont)
- J2: value Antenna -> External antenna
- K1: value AQY212SX -> AQY212SX (DNP); now not fitted
- R1: value 1k -> 10k; footprint Resistor_SMD:R_0603_1608Metric -> Resistor_THT:R_Axial_DIN0207_L6.3mm_D2.5mm_P2.54mm_Vertical
- R2: value 100 -> 1.1k; footprint Resistor_SMD:R_0603_1608Metric -> Resistor_THT:R_Axial_DIN0207_L6.3mm_D2.5mm_P2.54mm_Vertical
- R3, R4, R5: footprint Resistor_SMD:R_0603_1608Metric -> Resistor_THT:R_Axial_DIN0207_L6.3mm_D2.5mm_P2.54mm_Vertical
- R6: value 330 -> 330 (DNP); footprint Resistor_SMD:R_0603_1608Metric -> Resistor_THT:R_Axial_DIN0207_L6.3mm_D2.5mm_P2.54mm_Vertical; now not fitted
Connections:
- net +3V3: now also J3.1 (Pin_1), R8.2
- net CSW: now also K1.3 (A); no longer K1.4 (B)
- net DRV: now also JP1.2 (Pin_2); no longer C2.1, C3.1, C4.1, C5.1, K1.3 (A)
- net FSEL: now also J1.40 (Pin_40); no longer J1.37 (Pin_37)
- net GND: now also D2.1 (K), D3.1 (K), J3.4 (Pin_4), L1.2
- net I2C_SCL: now also J3.2 (Pin_2)
- net I2C_SDA: now also J3.3 (Pin_3)
- net SIGLED: now reaches J1.18 (Pin_18)
- net SIGLED: now also R7.2
- net ANT renamed ANT_X
- net ANT_X: now also JP2.2 (Pin_2)
- new net ANT_B: JP1.3 (Pin_3), L1.1
- new net EXT_IN: C2.1, C3.1, C4.1, C5.1, JP1.1 (Pin_1), JP2.1 (Pin_1), K1.4 (B)
- new net PWR_A: D3.2 (A), R8.1
- new net SIGLED_A: D2.2 (A), R7.1
- no-connect marks 38 -> 37
Other:
- note added: "JJY time unit 40/60kHz: connects to the Raspberry Pi 2x20 GPIO header with a ribbon or Dupont cable (J1, top centre)."
- note added: "L1 = on-board PCB spiral coil (2 layers, ~15uH, DC resistance ~4 ohm). Not resonant: the drive resistance is much larger than the coil reactance."
- note added: "U1A (always on) drives via R1 10k, U1B adds R2 1.1k in parallel: ratio = 1+R1/R2 = ~10:1 (-20dB). Keep R1 = ~9 x R2. Antenna current ~2mA."
- note added: "U2 DS3231SN + BT1 CR2032: on-board RTC (I2C pull-ups are on the Pi). J3 = I2C 16x2 LCD. D2 = signal LED (GPIO24)."
- note removed: "Band select: GPIO26 (FSEL). Low = 60kHz (default). High = K1 photo-MOS relay adds C7-C9 (9.1nF) -> 40kHz."
- note removed: "JJY HAT 40/60kHz (60kHz Hagane-yama default / 40kHz Ohtakadoya-yama), on-board RTC"
- note removed: "Series resonance: L(1mH) with C2+C3+C4 (+C5 trim) = 7.05nF -> 59.9kHz; with C7+C8+C9 (+9.1nF) = 16.15nF -> 39.6kHz. Measure L and tune C."
- note removed: "U1A (always on) drives via R1 1k, U1B adds R2 100R in parallel: (1k+Rcoil)/(91R+Rcoil) = ~10:1."
- note removed: "U2 DS3231SN + BT1 CR2032: on-board RTC (I2C pull-ups are on the Pi). Enable [rtc] in /etc/jjyd.toml."
- title: JJY HAT 40/60kHz for Raspberry Pi 4 -> JJY time unit 40/60kHz (cable to Raspberry Pi GPIO)
- moved on the sheet: J2

Commit message: Assemble K1 at JLCPCB and list DNP parts in the full BOM
- K1 (AQY212SX, C719754) is now an SMT part in the JLCPCB BOM/CPL
- Full BOM keeps DNP parts (C2-C5, C7-C9, R6) with a DNP column
- Docs updated accordingly; Gerber/BOM/CPL regenerated

Co-Authored-By: Claude Sonnet 5.5 <noreply@anthropic.com>
Parts:
- K1: value AQY212SX (DNP) -> AQY212SX; now fitted
Changed lines of the file:
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@@
     (pin "2")
     (instances (project "jjy-hat" (path "/40741956-28cf-5098-b1ad-9fedd8f61b8d" (reference "C9") (unit 1)))))
-  (symbol (lib_id "JJY:AQY212S") (at 203.2 228.6 0) (unit 1) (exclude_from_sim no) (in_bom yes) (on_board yes) (dnp yes) (property "Reference" "K1" (at 207.01 226.06 0) (effects (font (size 1.27 1.27)) (justify left))) (property "Value" "AQY212SX (DNP)" (at 207.01 228.6 0) (effects (font (size 1.27 1.27)) (justify left))) (property "Footprint" "Package_SO:SO-4_4.4x4.3mm_P2.54mm" (at 203.2 228.6 0) (effects (font (size 1.27 1.27)) hide)) (property "Datasheet" "~" (at 203.2 228.6 0) (effects (font (size 1.27 1.27)) hide))
+  (symbol (lib_id "JJY:AQY212S") (at 203.2 228.6 0) (unit 1) (exclude_from_sim no) (in_bom yes) (on_board yes) (dnp no) (property "Reference" "K1" (at 207.01 226.06 0) (effects (font (size 1.27 1.27)) (justify left))) (property "Value" "AQY212SX" (at 207.01 228.6 0) (effects (font (size 1.27 1.27)) (justify left))) (property "Footprint" "Package_SO:SO-4_4.4x4.3mm_P2.54mm" (at 203.2 228.6 0) (effects (font (size 1.27 1.27)) hide)) (property "Datasheet" "~" (at 203.2 228.6 0) (effects (font (size 1.27 1.27)) hide))
     (pin "1")
     (pin "2")
